File: hp5x21_rerouter/hp5x21_rerouter.kicad_pcb (KiCad board)
At the start: 2 copper layers, 10.6 x 21 mm, 3 parts, among them J1 Conn_01x08, J2 Conn_01x08, U2 74HC04

Commit message: Updated and released to JLCPCB
Connections:
- J1 pad 3: /C -> /~{C}_out
- J1 pad 4: /~{C}_out -> /C
Changed lines of the file:
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@@
 		(title "HP5X21 Rerouter")
 		(date "2025-03-29")
-		(rev "1.0")
+		(rev "1.1")
 		(company "alvarop.com")
 	)
@@
 			(at 0 2.33 0)
 			(layer "B.SilkS")
+			(hide yes)
 			(effects
 				(font
@@
 			)
 			(remove_unused_layers no)
-			(net 10 "/C")
+			(net 1 "/~{C}_out")
 			(pinfunction "Pin_3")
 			(pintype "passive")
@@
 			)
 			(remove_unused_layers no)
-			(net 1 "/~{C}_out")
+			(net 10 "/C")
 			(pinfunction "Pin_4")
 			(pintype "passive")
@@
 			(at 0 2.33 180)
 			(layer "B.SilkS")
-			(effects
-				(font
+			(hide yes)
+			(effects
+				(font
