File: hp5x21_rerouter/hp5x21_rerouter.kicad_sch (KiCad schematic)
At the start: 3 parts, among them J1 Conn_01x08, J2 Conn_01x08, U2 74HC04

Commit message: Updated and released to JLCPCB
Connections:
- net C: now also J1.4 (Pin_4); no longer J1.3 (Pin_3)
- net ~{C}_out: now also J1.3 (Pin_3); no longer J1.4 (Pin_4)
Changed lines of the file:
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@@
 	)
 	(label "~{C}_out"
-		(at 86.36 111.76 0)
+		(at 86.36 109.22 0)
 		(effects
 			(font
@@
 	)
 	(label "C"
-		(at 86.36 109.22 0)
+		(at 86.36 111.76 0)
 		(effects
 			(font
